File: hardware/KiCad/blinky_badge_light/blinky_badge_light.kicad_sch (KiCad schematic)
At the start: 9 parts, among them U1 ESP32-S3-WROOM-1

Commit message: updates to hardware schematic
Parts:
- added C38: 100nF, Capacitor_SMD:C_0402_1005Metric, symbol Device:C
- added C39: 22µF, Capacitor_SMD:C_0201_0603Metric, symbol Device:C
- added C40: 1µF, Capacitor_SMD:C_0603_1608Metric, symbol Device:C
- C31: footprint Capacitor_SMD:C_0402_1005Metric -> Resistor_SMD:R_0402_1005Metric
- U1: footprint PCM_Espressif:ESP32-S3-WROOM-1 -> RF_Module:ESP32-S3-WROOM-1
Connections:
- net 3.3V Power: now also R11.2, C38.2, C39.1; no longer R11.1
- net ESP32 Reset: now also R11.1, U1.3 (EN), C40.2
- net GND: now also C31.1, C38.1, C39.2, C40.1
Other:
- moved on the sheet: R11

Commit message: hardware updates, gitignore to ignore backups
Parts:
- TOUCH_1, TOUCH_2, TOUCH_3, TOUCH_4: footprint TestPoint:TestPoint_Pad_D4.0mm -> footprints:TestPoint_Pad_D12.0mm
Changed lines of the file:
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@@
 			)
 		)
-		(property "Footprint" "TestPoint:TestPoint_Pad_D4.0mm"
+		(property "Footprint" "footprints:TestPoint_Pad_D12.0mm"
 			(at 234.95 100.33 0)
 			(effects
@@
 			)
 		)
-		(property "Footprint" "TestPoint:TestPoint_Pad_D4.0mm"
+		(property "Footprint" "footprints:TestPoint_Pad_D12.0mm"
 			(at 234.95 107.95 0)
 			(effects
@@
 			)
 		)
-		(property "Footprint" "TestPoint:TestPoint_Pad_D4.0mm"
+		(property "Footprint" "footprints:TestPoint_Pad_D12.0mm"
 			(at 234.95 92.71 0)
 			(effects
@@
 			)
 		)
-		(property "Footprint" "TestPoint:TestPoint_Pad_D4.0mm"
+		(property "Footprint" "footprints:TestPoint_Pad_D12.0mm"
 			(at 234.95 85.09 0)
 			(effects

Commit message: stuff from today
Parts:
- C39: footprint Capacitor_SMD:C_0201_0603Metric -> Capacitor_SMD:C_0603_1608Metric
Changed lines of the file:
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@@
 			)
 		)
-		(property "Footprint" "Capacitor_SMD:C_0201_0603Metric"
+		(property "Footprint" "Capacitor_SMD:C_0603_1608Metric"
 			(at 132.08 29.5148 0)
 			(effects

Commit message: fix some stuff with the footprints, rearrange some things
Parts:
- C31: footprint Resistor_SMD:R_0402_1005Metric -> Capacitor_SMD:C_0402_1005Metric
- TOUCH_4: footprint footprints:TestPoint_Pad_D12.0mm -> TestPoint:TestPoint_Pad_D4.0mm
Changed lines of the file:
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@@
 			)
 		)
-		(property "Footprint" "footprints:TestPoint_Pad_D12.0mm"
+		(property "Footprint" "TestPoint:TestPoint_Pad_D4.0mm"
 			(at 234.95 107.95 0)
 			(effects
@@
 			)
 		)
-		(property "Footprint" "Resistor_SMD:R_0402_1005Metric"
+		(property "Footprint" "Capacitor_SMD:C_0402_1005Metric"
 			(at 82.8548 59.69 0)
 			(effects

Commit message: pad 4 is now stop sign shaped since its the off button
Parts:
- TOUCH_4: footprint TestPoint:TestPoint_Pad_D4.0mm -> footprints:Touch_Pad_StopSign_6mm
Changed lines of the file:
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@@
 			)
 		)
-		(property "Footprint" "TestPoint:TestPoint_Pad_D4.0mm"
+		(property "Footprint" "footprints:Touch_Pad_StopSign_6mm"
 			(at 234.95 107.95 0)
 			(effects

Commit message: clean up labels on the back
Parts:
- U1: footprint RF_Module:ESP32-S3-WROOM-1 -> footprints:ESP32-S3-WROOM-1 - no antenna keep out
Changed lines of the file:
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@@
 			)
 		)
-		(property "Footprint" "RF_Module:ESP32-S3-WROOM-1"
+		(property "Footprint" "footprints:ESP32-S3-WROOM-1 - no antenna keep out"
 			(at 148.59 143.51 0)
 			(effects

Commit message: revert last changes so I can merge other branch in
Parts:
- U1: footprint footprints:ESP32-S3-WROOM-1 - no antenna keep out -> RF_Module:ESP32-S3-WROOM-1
Changed lines of the file:
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@@
 			)
 		)
-		(property "Footprint" "footprints:ESP32-S3-WROOM-1 - no antenna keep out"
+		(property "Footprint" "RF_Module:ESP32-S3-WROOM-1"
 			(at 148.59 143.51 0)
 			(effects

Commit message: update with routing
Connections:
- net at TOUCH_3.1: now also U1.15 (GPIO3/TOUCH3/ADC1_CH2); no longer U1.5 (GPIO5/TOUCH5/ADC1_CH4)
- net at TOUCH_4.1: now also U1.4 (GPIO4/TOUCH4/ADC1_CH3); no longer U1.6 (GPIO6/TOUCH6/ADC1_CH5)
- net at TOUCH_2.1: now also U1.6 (GPIO6/TOUCH6/ADC1_CH5); no longer U1.4 (GPIO4/TOUCH4/ADC1_CH3)
- net at TOUCH_1.1: now also U1.5 (GPIO5/TOUCH5/ADC1_CH4); no longer U1.15 (GPIO3/TOUCH3/ADC1_CH2)
Other:
- moved on the sheet: TOUCH_1, TOUCH_2, TOUCH_3, TOUCH_4
Changed lines of the file:
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@@
-	(wire
-		(pts
-			(xy 215.9 107.95) (xy 229.87 107.95)
-		)
-		(stroke
-			(width 0)
-			(type default)
-		)
-	)
 	(wire
 		(pts
@@
 	(wire
 		(pts
-			(xy 229.87 100.33) (xy 219.71 100.33)
-		)
-		(stroke
-			(width 0)
-			(type default)
-		)
-	)
-	(wire
-		(pts
-			(xy 229.87 85.09) (xy 226.06 85.09)
-		)
-		(stroke
-			(width 0)
-			(type default)
-		)
-	)
-	(wire
-		(pts
 			(xy 83.82 59.69) (xy 92.71 59.69)
 		)
@@
 	(wire
 		(pts
-			(xy 229.87 92.71) (xy 223.52 92.71)
-		)
-		(stroke
-			(width 0)
-			(type default)
-		)
-	)
-	(wire
-		(pts
 			(xy 228.6 68.58) (xy 224.79 68.58)
 		)
@@
 	(wire
 		(pts
+			(xy 223.52 92.71) (xy 231.14 92.71)
+		)
+		(stroke
+			(width 0)
+			(type default)
+		)
+	)
+	(wire
+		(pts
 			(xy 124.46 30.48) (xy 124.46 40.64)
 		)
@@
 	(wire
 		(pts
+			(xy 215.9 107.95) (xy 219.71 107.95)
+		)
+		(stroke
+			(width 0)
+			(type default)
+		)
+	)
+	(wire
+		(pts
 			(xy 101.6 45.72) (xy 92.71 45.72)
 		)
@@
 	(wire
 		(pts
+			(xy 226.06 85.09) (xy 231.14 85.09)
+		)
+		(stroke
+			(width 0)
+			(type default)
+		)
+	)
+	(wire
+		(pts
 			(xy 198.12 68.58) (xy 198.12 74.93)
 		)
@@
 		(pts
 			(xy 124.46 45.72) (xy 109.22 45.72)
+		)
+		(stroke
+			(width 0)
+			(type default)
+		)
+	)
+	(wire
+		(pts
+			(xy 219.71 100.33) (xy 231.14 100.33)
 		)
 		(stroke
@@
 	(symbol
 		(lib_id "Connector:TestPoint")
-		(at 229.87 100.33 0)
+		(at 231.14 85.09 0)
 		(unit 1)
 		(exclude_from_sim no)
@@
 		(fields_autoplaced yes)
 		(property "Reference" "TOUCH_3"
-			(at 232.41 95.7579 0)
+			(at 233.68 80.5179 0)
 			(effects
 				(font
@@
 		)
 		(property "Value" "TestPoint"
-			(at 232.41 98.2979 0)
+			(at 233.68 83.0579 0)
 			(effects
 				(font
@@
 		)
 		(property "Footprint" "footprints:TestPoint_Pad_D12.0mm"
-			(at 234.95 100.33 0)
+			(at 236.22 85.09 0)
 			(effects
 				(font
@@
 		)
 		(property "Datasheet" "~"
-			(at 234.95 100.33 0)
+			(at 236.22 85.09 0)
 			(effects
 				(font
@@
 		)
 		(property "Description" "test point"
-			(at 229.87 100.33 0)
+			(at 231.14 85.09 0)
 			(effects
 				(font
@@
 	(symbol
 		(lib_id "Connector:TestPoint")
-		(at 229.87 107.95 0)
+		(at 231.14 92.71 0)
 		(unit 1)
 		(exclude_from_sim no)
@@
 		(fields_autoplaced yes)
 		(property "Reference" "TOUCH_4"
-			(at 232.41 103.3779 0)
+			(at 233.68 88.1379 0)
 			(effects
 				(font
@@
 		)
 		(property "Value" "TestPoint"
-			(at 232.41 105.9179 0)
+			(at 233.68 90.6779 0)
 			(effects
 				(font
@@
 		)
 		(property "Footprint" "footprints:Touch_Pad_StopSign_6mm"
-			(at 234.95 107.95 0)
+			(at 236.22 92.71 0)
 			(effects
 				(font
@@
 		)
 		(property "Datasheet" "~"
-			(at 234.95 107.95 0)
+			(at 236.22 92.71 0)
 			(effects
 				(font
@@
 		)
 		(property "Description" "test point"
-			(at 229.87 107.95 0)
+			(at 231.14 92.71 0)
 			(effects
 				(font
@@
 	(symbol
 		(lib_id "Connector:TestPoint")
-		(at 229.87 92.71 0)
+		(at 219.71 107.95 0)
 		(unit 1)
 		(exclude_from_sim no)
@@
 		(fields_autoplaced yes)
 		(property "Reference" "TOUCH_2"
-			(at 232.41 88.1379 0)
+			(at 222.25 103.3779 0)
 			(effects
 				(font
@@
 		)
 		(property "Value" "TestPoint"
-			(at 232.41 90.6779 0)
+			(at 222.25 105.9179 0)
 			(effects
 				(font
@@
 		)
 		(property "Footprint" "footprints:TestPoint_Pad_D12.0mm"
-			(at 234.95 92.71 0)
+			(at 224.79 107.95 0)
 			(effects
 				(font
@@
 		)
 		(property "Datasheet" "~"
-			(at 234.95 92.71 0)
+			(at 224.79 107.95 0)
 			(effects
 				(font
@@
 		)
 		(property "Description" "test point"
-			(at 229.87 92.71 0)
+			(at 219.71 107.95 0)
 			(effects
 				(font
@@
 	(symbol
 		(lib_id "Connector:TestPoint")
-		(at 229.87 85.09 0)
+		(at 231.14 100.33 0)
 		(unit 1)
 		(exclude_from_sim no)
@@
 		(fields_autoplaced yes)
 		(property "Reference" "TOUCH_1"
-			(at 232.41 80.5179 0)
+			(at 233.68 95.7579 0)
 			(effects
 				(font
@@
 		)
 		(property "Value" "TestPoint"
-			(at 232.41 83.0579 0)
+			(at 233.68 98.2979 0)
 			(effects
 				(font
@@
 		)
 		(property "Footprint" "footprints:TestPoint_Pad_D12.0mm"
-			(at 234.95 85.09 0)
+			(at 236.22 100.33 0)
 			(effects
 				(font
@@
 		)
 		(property "Datasheet" "~"
-			(at 234.95 85.09 0)
+			(at 236.22 100.33 0)
 			(effects
 				(font
@@
 		)
 		(property "Description" "test point"
-			(at 229.87 85.09 0)
-			(effects
-				(font
+			(at 231.14 100.33 0)
+			(effects
+				(font
